Commit message: changed to xz plane
However, the gcD_test and WBC_CTRL not work

File: five_link_walker.urdf (robot description, URDF)
Before this commit: robot five_link_walker, 10 links, 9 joints
Links:
- removed link y_prismatic
- added link x_prismatic, mass 0.01
Joints:
- removed joint y_to_world
- added joint x_to_world: type prismatic, parent world, child x_prismatic, origin xyz=0 0 0 rpy=0 0 0, axis 1 0 0, limit lower=-10 upper=10 effort=0.0 velocity=1000.0
- joint q1_left: axis 1 0 0 -> 0 1 0
- joint q1_right: axis 1 0 0 -> 0 1 0
- joint q2_left: axis 1 0 0 -> 0 1 0
- joint q2_right: axis 1 0 0 -> 0 1 0
- joint torso_to_z: axis 1 0 0 -> 0 1 0
- joint z_to_y: parent y_prismatic -> x_prismatic
