Commit message: HZD optimization evolve
Tested a new HZD reference traj framework and parameter in `newVCwalkTest.py`

added BezierUtil

added Uilt control components in rabbit ctrl:
- auto_camera
- circulatePosition

File: five_link_walker_xz.urdf (robot description, URDF)
Before this commit: robot five_link_walker, 10 links, 9 joints
Joints:
- joint x_to_world: limit lower=-10 upper=10 effort=0.0 velocity=1000.0 -> lower=-20 upper=20 effort=0.0 velocity=1000.0
